File: SmallKat Jumbo Motherboard.sch (KiCad schematic (older format))
At the start: 49 parts, among them IC1 TPS562201DDCR, IC2 TPS562201DDCR, J1 Conn_01x06_Male, J10 Conn_01x06_Male, J11 Conn_01x06_Male, J12 Conn_01x04_Male, J13 Conn_01x02_Male, J14 Conn_01x04_Male, J15 Conn_01x04_Male, J16 Conn_01x06_Male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

Commit message: Changed footprints
Parts:
- removed Y1: 32MHZ, Crystal:Crystal_SMD_2016-4Pin_2.0x1.6mm, symbol Device:Crystal_GND24
- added Y1: 32.768khz, Crystal:Crystal_SMD_2012-2Pin_2.0x1.2mm, symbol Device:Crystal
- C1: value C -> 1UF
- C10, C11, C16, C17: value C -> 0.1UF
- C12, C13, C6, C7: value C -> 22UF
- C14, C15, C8, C9: value C -> 10UF
- C2, C3, C4, C5: value C -> 10PF
- D1, D2: value D -> 641-1675-1-ND
- L1, L2: value L -> 4.7UH
- R1, R2, R3, R5, R6: value R -> 10K
- R4, R7: value R -> 33.2K
Changed lines of the file:
@@
 P 3400 1500
 F 0 "R1" V 3193 1500 50  0000 C CNN
-F 1 "R" V 3284 1500 50  0000 C CNN
+F 1 "10K" V 3284 1500 50  0000 C CNN
 F 2 "Resistor_SMD:R_0402_1005Metric" V 3330 1500 50  0001 C CNN
 F 3 "~" H 3400 1500 50  0001 C CNN
@@
 	10000 1000 15500 1000
 $Comp
-L Device:Crystal_GND24 Y1
-U 1 1 5B785BE1
-P 10750 4450
-F 0 "Y1" H 11050 4650 50  0000 L CNN
-F 1 "32MHZ" H 11000 4300 50  0000 L CNN
-F 2 "Crystal:Crystal_SMD_2016-4Pin_2.0x1.6mm" H 10750 4450 50  0001 C CNN
-F 3 "~" H 10750 4450 50  0001 C CNN
-	1    10750 4450
-	1    0    0    -1
-$EndComp
-$Comp
 L Device:Crystal_GND24 Y2
 U 1 1 5B785C94
@@
 Text GLabel 12050 4450 2    50   Input ~ 0
 OSCOUT
-$Comp
-L power:GND #PWR0129
-U 1 1 5B786107
-P 10750 4650
-F 0 "#PWR0129" H 10750 4400 50  0001 C CNN
-F 1 "GND" H 10755 4477 50  0000 C CNN
-F 2 "" H 10750 4650 50  0001 C CNN
-F 3 "" H 10750 4650 50  0001 C CNN
-	1    10750 4650
-	1    0    0    -1
-$EndComp
-$Comp
-L power:GND #PWR0130
-U 1 1 5B786159
-P 10750 4250
-F 0 "#PWR0130" H 10750 4000 50  0001 C CNN
-F 1 "GND" H 10755 4077 50  0000 C CNN
-F 2 "" H 10750 4250 50  0001 C CNN
-F 3 "" H 10750 4250 50  0001 C CNN
-	1    10750 4250
-	-1   0    0    1
-$EndComp
 $Comp
 L power:GND #PWR0131
@@
 P 6400 750
 F 0 "C1" V 6148 750 50  0000 C CNN
-F 1 "C" V 6239 750 50  0000 C CNN
+F 1 "1UF" V 6239 750 50  0000 C CNN
 F 2 "Capacitor_SMD:C_0402_1005Metric" H 6438 600 50  0001 C CNN
 F 3 "~" H 6400 750 50  0001 C CNN
@@
 P 12050 4600
 F 0 "C5" H 12165 4646 50  0000 L CNN
-F 1 "C" H 12165 4555 50  0000 L CNN
+F 1 "10PF" H 12165 4555 50  0000 L CNN
 F 2 "Capacitor_SMD:C_0402_1005Metric" H 12088 4450 50  0001 C CNN
 F 3 "~" H 12050 4600 50  0001 C CNN
@@
 P 11750 4600
 F 0 "C4" H 11865 4646 50  0000 L CNN
-F 1 "C" H 11865 4555 50  0000 L CNN
+F 1 "10PF" H 11865 4555 50  0000 L CNN
 F 2 "Capacitor_SMD:C_0402_1005Metric" H 11788 4450 50  0001 C CNN
 F 3 "~" H 11750 4600 50  0001 C CNN
@@
 P 10900 4600
 F 0 "C3" H 11015 4646 50  0000 L CNN
-F 1 "C" H 11015 4555 50  0000 L CNN
+F 1 "10PF" H 11015 4555 50  0000 L CNN
 F 2 "Capacitor_SMD:C_0402_1005Metric" H 10938 4450 50  0001 C CNN
 F 3 "~" H 10900 4600 50  0001 C CNN
@@
 P 10600 4600
 F 0 "C2" H 10715 4646 50  0000 L CNN
-F 1 "C" H 10715 4555 50  0000 L CNN
+F 1 "10PF" H 10715 4555 50  0000 L CNN
 F 2 "Capacitor_SMD:C_0402_1005Metric" H 10638 4450 50  0001 C CNN
 F 3 "~" H 10600 4600 50  0001 C CNN
@@
 U 1 1 5B78BA0C
 P 11700 6200
-F 0 "R3" V 11493 6200 50  0000 C CNN
-F 1 "R" V 11584 6200 50  0000 C CNN
+F 0 "R3" V 11650 6350 50  0000 C CNN
+F 1 "10K" V 11700 6200 50  0000 C CNN
 F 2 "Resistor_SMD:R_0402_1005Metric" V 11630 6200 50  0001 C CNN
 F 3 "~" H 11700 6200 50  0001 C CNN
@@
 U 1 1 5B78BADF
 P 11700 6300
-F 0 "R4" V 11493 6300 50  0000 C CNN
-F 1 "R" V 11584 6300 50  0000 C CNN
+F 0 "R4" V 11750 6450 50  0000 C CNN
+F 1 "33.2K" V 11700 6300 50  0000 C CNN
 F 2 "Resistor_SMD:R_0402_1005Metric" V 11630 6300 50  0001 C CNN
 F 3 "~" H 11700 6300 50  0001 C CNN
@@
 P 11550 6450
 F 0 "R2" H 11620 6496 50  0000 L CNN
-F 1 "R" H 11620 6405 50  0000 L CNN
+F 1 "10K" H 11620 6405 50  0000 L CNN
 F 2 "Resistor_SMD:R_0402_1005Metric" V 11480 6450 50  0001 C CNN
 F 3 "~" H 11550 6450 50  0001 C CNN
@@
 U 1 1 5B78CA2E
 P 10300 6450
-F 0 "C10" H 10415 6496 50  0000 L CNN
-F 1 "C" H 10415 6405 50  0000 L CNN
+F 0 "C10" H 10300 6550 50  0000 L CNN
+F 1 "0.1UF" H 10300 6350 50  0000 L CNN
 F 2 "Capacitor_SMD:C_0402_1005Metric" H 10338 6300 50  0001 C CNN
 F 3 "~" H 10300 6450 50  0001 C CNN
@@
 U 1 1 5B78CABD
 P 10100 6450
-F 0 "C9" H 10215 6496 50  0000 L CNN
-F 1 "C" H 10215 6405 50  0000 L CNN
+F 0 "C9" H 10150 6550 50  0000 L CNN
+F 1 "10UF" H 10100 6350 50  0000 L CNN
 F 2 "Capacitor_SMD:C_0402_1005Metric" H 10138 6300 50  0001 C CNN
 F 3 "~" H 10100 6450 50  0001 C CNN
@@
 U 1 1 5B78CB3D
 P 9900 6450
-F 0 "C8" H 10015 6496 50  0000 L CNN
-F 1 "C" H 10015 6405 50  0000 L CNN
+F 0 "C8" H 9950 6550 50  0000 L CNN
+F 1 "10UF" H 9900 6350 50  0000 L CNN
 F 2 "Capacitor_SMD:C_0402_1005Metric" H 9938 6300 50  0001 C CNN
 F 3 "~" H 9900 6450 50  0001 C CNN
@@
 P 9800 6100
 F 0 "L1" V 9990 6100 50  0000 C CNN
-F 1 "L" V 9899 6100 50  0000 C CNN
+F 1 "4.7UH" V 9899 6100 50  0000 C CNN
 F 2 "Inductor_SMD:L_1206_3216Metric" H 9800 6100 50  0001 C CNN
 F 3 "~" H 9800 6100 50  0001 C CNN
@@
 U 1 1 5B790039
 P 9550 6250
-F 0 "C7" H 9665 6296 50  0000 L CNN
-F 1 "C" H 9665 6205 50  0000 L CNN
+F 0 "C7" H 9650 6350 50  0000 L CNN
+F 1 "22UF" H 9650 6250 50  0000 L CNN
 F 2 "Capacitor_SMD:C_0402_1005Metric" H 9588 6100 50  0001 C CNN
 F 3 "~" H 9550 6250 50  0001 C CNN
@@
 U 1 1 5B7900C6
 P 9350 6250
-F 0 "C6" H 9465 6296 50  0000 L CNN
-F 1 "C" H 9465 6205 50  0000 L CNN
+F 0 "C6" H 9100 6300 50  0000 L CNN
+F 1 "22UF" H 9050 6200 50  0000 L CNN
 F 2 "Capacitor_SMD:C_0402_1005Metric" H 9388 6100 50  0001 C CNN
 F 3 "~" H 9350 6250 50  0001 C CNN
@@
 P 10850 5650
 F 0 "C11" V 10598 5650 50  0000 C CNN
-F 1 "C" V 10689 5650 50  0000 C CNN
+F 1 "0.1UF" V 10689 5650 50  0000 C CNN
 F 2 "Capacitor_SMD:C_0402_1005Metric" H 10888 5500 50  0001 C CNN
 F 3 "~" H 10850 5650 50  0001 C CNN
@@
 P 9000 6100
 F 0 "D2" H 9000 6316 50  0000 C CNN
-F 1 "D" H 9000 6225 50  0000 C CNN
+F 1 "641-1675-1-ND" H 9000 6225 50  0000 C CNN
 F 2 "Diode_SMD:D_0402_1005Metric" H 9000 6100 50  0001 C CNN
-F 3 "~" H 9000 6100 50  0001 C CNN
+F 3 "CDBQR0130L-HF" H 9000 6100 50  0001 C CNN
 	1    9000 6100
 	1    0    0    -1
@@
 U 1 1 5B795FA0
 P 11600 7650
-F 0 "R6" V 11393 7650 50  0000 C CNN
-F 1 "R" V 11484 7650 50  0000 C CNN
+F 0 "R6" V 11550 7800 50  0000 C CNN
+F 1 "10K" V 11600 7650 50  0000 C CNN
 F 2 "Resistor_SMD:R_0402_1005Metric" V 11530 7650 50  0001 C CNN
 F 3 "~" H 11600 7650 50  0001 C CNN
@@
 U 1 1 5B795FA7
 P 11600 7750
-F 0 "R7" V 11393 7750 50  0000 C CNN
-F 1 "R" V 11484 7750 50  0000 C CNN
+F 0 "R7" V 11650 7900 50  0000 C CNN
+F 1 "33.2K" V 11600 7750 50  0000 C CNN
 F 2 "Resistor_SMD:R_0402_1005Metric" V 11530 7750 50  0001 C CNN
 F 3 "~" H 11600 7750 50  0001 C CNN
@@
 P 11450 7900
 F 0 "R5" H 11520 7946 50  0000 L CNN
-F 1 "R" H 11520 7855 50  0000 L CNN
+F 1 "10K" H 11520 7855 50  0000 L CNN
 F 2 "Resistor_SMD:R_0402_1005Metric" V 11380 7900 50  0001 C CNN
 F 3 "~" H 11450 7900 50  0001 C CNN
@@
 P 10200 7900
 F 0 "C16" H 10315 7946 50  0000 L CNN
-F 1 "C" H 10315 7855 50  0000 L CNN
+F 1 "0.1UF" H 10315 7855 50  0000 L CNN
 F 2 "Capacitor_SMD:C_0402_1005Metric" H 10238 7750 50  0001 C CNN
 F 3 "~" H 10200 7900 50  0001 C CNN
@@
 P 10000 7900
 F 0 "C15" H 10115 7946 50  0000 L CNN
-F 1 "C" H 10115 7855 50  0000 L CNN
+F 1 "10UF" H 10115 7855 50  0000 L CNN
 F 2 "Capacitor_SMD:C_0402_1005Metric" H 10038 7750 50  0001 C CNN
 F 3 "~" H 10000 7900 50  0001 C CNN
@@
 P 9800 7900
 F 0 "C14" H 9915 7946 50  0000 L CNN
-F 1 "C" H 9915 7855 50  0000 L CNN
+F 1 "10UF" H 9915 7855 50  0000 L CNN
 F 2 "Capacitor_SMD:C_0402_1005Metric" H 9838 7750 50  0001 C CNN
 F 3 "~" H 9800 7900 50  0001 C CNN
@@
 P 9700 7550
 F 0 "L2" V 9890 7550 50  0000 C CNN
-F 1 "L" V 9799 7550 50  0000 C CNN
+F 1 "4.7UH" V 9799 7550 50  0000 C CNN
 F 2 "Inductor_SMD:L_1206_3216Metric" H 9700 7550 50  0001 C CNN
 F 3 "~" H 9700 7550 50  0001 C CNN
@@
 P 9450 7700
 F 0 "C13" H 9565 7746 50  0000 L CNN
-F 1 "C" H 9565 7655 50  0000 L CNN
+F 1 "22UF" H 9565 7655 50  0000 L CNN
 F 2 "Capacitor_SMD:C_0402_1005Metric" H 9488 7550 50  0001 C CNN
 F 3 "~" H 9450 7700 50  0001 C CNN
@@
 P 9250 7700
 F 0 "C12" H 9365 7746 50  0000 L CNN
-F 1 "C" H 9365 7655 50  0000 L CNN
+F 1 "22UF" H 9365 7655 50  0000 L CNN
 F 2 "Capacitor_SMD:C_0402_1005Metric" H 9288 7550 50  0001 C CNN
 F 3 "~" H 9250 7700 50  0001 C CNN
@@
 P 10750 7100
 F 0 "C17" V 10498 7100 50  0000 C CNN
-F 1 "C" V 10589 7100 50  0000 C CNN
+F 1 "0.1UF" V 10589 7100 50  0000 C CNN
 F 2 "Capacitor_SMD:C_0402_1005Metric" H 10788 6950 50  0001 C CNN
 F 3 "~" H 10750 7100 50  0001 C CNN
@@
 P 8900 7550
 F 0 "D1" H 8900 7766 50  0000 C CNN
-F 1 "D" H 8900 7675 50  0000 C CNN
+F 1 "641-1675-1-ND" H 8900 7675 50  0000 C CNN
 F 2 "Diode_SMD:D_0402_1005Metric" H 8900 7550 50  0001 C CNN
-F 3 "~" H 8900 7550 50  0001 C CNN
+F 3 "CDBQR0130L-HF" H 8900 7550 50  0001 C CNN
 	1    8900 7550
 	1    0    0    -1
@@
 Text GLabel 4450 5900 0    50   Input ~ 0
 CS5_2
+$Comp
+L Device:Crystal Y1
+U 1 1 5B836102
+P 10750 4450
+F 0 "Y1" H 10750 4718 50  0000 C CNN
+F 1 "32.768khz" H 10750 4627 50  0000 C CNN
+F 2 "Crystal:Crystal_SMD_2012-2Pin_2.0x1.2mm" H 10750 4450 50  0001 C CNN
+F 3 "~" H 10750 4450 50  0001 C CNN
+	1    10750 4450
+	1    0    0    -1
+$EndComp
 $EndSCHEMATC

Commit message: fixed pinout
Parts:
- removed J12: Conn_01x04_Male, Connector_Molex:Molex_CLIK-Mate_502443-0470_1x04-1MP_P2.00mm_Vertical, symbol Connector:Conn_01x04_Male
- added J12: Conn_01x05_Male, Connector_Molex:Molex_CLIK-Mate_502443-0570_1x05-1MP_P2.00mm_Vertical, symbol Connector:Conn_01x05_Male
Connections:
- net labels added: NRST
Changed lines of the file:
@@
 SWCLK
-$Comp
-L Connector:Conn_01x04_Male J12
-U 1 1 5B78655A
-P 15050 3200
-F 0 "J12" V 15110 3340 50  0000 L CNN
-F 1 "Conn_01x04_Male" V 15000 2850 50  0000 L CNN
-F 2 "Connector_Molex:Molex_CLIK-Mate_502443-0470_1x04-1MP_P2.00mm_Vertical" H 15050 3200 50  0001 C CNN
-F 3 "~" H 15050 3200 50  0001 C CNN
-	1    15050 3200
-	0    1    1    0
-$EndComp
 $Comp
 L power:GND #PWR0133
@@
 $EndComp
 $Comp
-L power:+BATT #PWR0141
-U 1 1 5B78BCDD
-P 11850 6300
-F 0 "#PWR0141" H 11850 6150 50  0001 C CNN
-F 1 "+BATT" V 11865 6428 50  0000 L CNN
-F 2 "" H 11850 6300 50  0001 C CNN
-F 3 "" H 11850 6300 50  0001 C CNN
-	1    11850 6300
-	0    1    1    0
-$EndComp
-$Comp
 L power:+BATT #PWR0142
 U 1 1 5B78BD67
@@
 F 3 "" H 11750 7650 50  0001 C CNN
 	1    11750 7650
-	0    1    1    0
-$EndComp
-$Comp
-L power:+5V #PWR0152
-U 1 1 5B799D73
-P 11750 7750
-F 0 "#PWR0152" H 11750 7600 50  0001 C CNN
-F 1 "+5V" V 11765 7878 50  0000 L CNN
-F 2 "" H 11750 7750 50  0001 C CNN
-F 3 "" H 11750 7750 50  0001 C CNN
-	1    11750 7750
 	0    1    1    0
 $EndComp
@@
 	1    0    0    -1
 $EndComp
+$Comp
+L power:+3.3V #PWR0129
+U 1 1 5BADB086
+P 11850 6300
+F 0 "#PWR0129" H 11850 6150 50  0001 C CNN
+F 1 "+3.3V" V 11865 6428 50  0000 L CNN
+F 2 "" H 11850 6300 50  0001 C CNN
+F 3 "" H 11850 6300 50  0001 C CNN
+	1    11850 6300
+	0    1    1    0
+$EndComp
+$Comp
+L power:+3.3V #PWR0130
+U 1 1 5BADB16C
+P 11750 7750
+F 0 "#PWR0130" H 11750 7600 50  0001 C CNN
+F 1 "+3.3V" V 11765 7878 50  0000 L CNN
+F 2 "" H 11750 7750 50  0001 C CNN
+F 3 "" H 11750 7750 50  0001 C CNN
+	1    11750 7750
+	0    1    1    0
+$EndComp
+Text GLabel 4450 1200 0    50   Input ~ 0
+NRST
+$Comp
+L Connector:Conn_01x05_Male J12
+U 1 1 5BADBF81
+P 15050 3200
+F 0 "J12" V 15110 3440 50  0000 L CNN
+F 1 "Conn_01x05_Male" V 15201 3440 50  0000 L CNN
+F 2 "Connector_Molex:Molex_CLIK-Mate_502443-0570_1x05-1MP_P2.00mm_Vertical" H 15050 3200 50  0001 C CNN
+F 3 "~" H 15050 3200 50  0001 C CNN
+	1    15050 3200
+	0    1    1    0
+$EndComp
+Text GLabel 15250 3400 3    50   Input ~ 0
+NRST
 $EndSCHEMATC

Commit message: Rev 2
Parts:
- removed C10, C11: 0.1UF, Capacitor_SMD:C_0402_1005Metric, symbol Device:C
- removed C6, C7: 22UF, Capacitor_SMD:C_0402_1005Metric, symbol Device:C
- removed C8, C9: 10UF, Capacitor_SMD:C_0402_1005Metric, symbol Device:C
- removed D1, D2: 641-1675-1-ND, Diode_SMD:D_0402_1005Metric, symbol Device:D
- removed IC1: TPS562201DDCR, TPS562201DDCR:SOT95P280X110-6N, symbol TPS562201DDCR:TPS562201DDCR
- removed J10, J11, J8, J9: Conn_01x06_Male, Connector_Molex:Molex_CLIK-Mate_502443-0670_1x06-1MP_P2.00mm_Vertical, symbol Connector:Conn_01x06_Male
- removed J12: Conn_01x05_Male, Connector_Molex:Molex_CLIK-Mate_502443-0570_1x05-1MP_P2.00mm_Vertical, symbol Connector:Conn_01x05_Male
- removed J13: Conn_01x02_Male, Connector_Molex:Molex_CLIK-Mate_502443-0270_1x02-1MP_P2.00mm_Vertical, symbol Connector:Conn_01x02_Male
- removed L1: 4.7UH, Inductor_SMD:L_1206_3216Metric, symbol Device:L
- removed U1: STM32H753IITx, Package_QFP:LQFP-176_24x24mm_P0.5mm, symbol MCU_ST_STM32H7:STM32H753IITx
- added C18, C19, C20, C21, C22, C23: 0.1uF, Capacitor_SMD:C_0402_1005Metric, symbol Device:C
- added D1, D2, D3: LED, LED_SMD:LED_0603_1608Metric, symbol Device:LED
- added FB1: Ferrite_Bead, Inductor_SMD:L_0805_2012Metric, symbol Device:Ferrite_Bead
- added H1, H2, H3: MountingHole, MountingHole:MountingHole_3.2mm_M3, symbol Mechanical:MountingHole
- added J10, J9: Conn_01x04_Male, Connector_Molex:Molex_CLIK-Mate_502443-0470_1x04-1MP_P2.00mm_Vertical, symbol Connector:Conn_01x04_Male
- added J8: PRT-10474, PRT-10474:SHDR2W320P716_1X2_1574X813X1588P, symbol PRT-10474:PRT-10474
- added R10: 10k, Resistor_SMD:R_0402_1005Metric, symbol Device:R
- added R11, R12, R8, R9: 33R, Resistor_SMD:R_0402_1005Metric, symbol Device:R
- added U1: STM32H743VITx, Package_QFP:LQFP-100_14x14mm_P0.5mm, symbol MCU_ST_STM32H7:STM32H743VITx
- C1: value 1UF -> 0.1uF
- C12, C13, C14, C15, C16: footprint Capacitor_SMD:C_0402_1005Metric -> Capacitor_SMD:C_0805_2012Metric
- L2: footprint Inductor_SMD:L_1206_3216Metric -> Inductor_SMD:L_0805_2012Metric_Pad1.15x1.40mm_HandSolder; Part Number (none) -> 74479776247
- R1, R5: value 10K -> 10k
- R2, R3: value 10K -> 330R
- R4: value 33.2K -> 330R
- R7: value 33.2K -> 33.2k
Connections:
- net labels added: CS1, CS6_HEAD, CS6_TAIL, IMU1_CS, IMU2_CS, LED1, LED2, LED3, MCU_GND, USB_FS_N, USB_FS_P, USB_HS_N, USB_HS_P
- net labels removed: CS1_1, CS1_2, CS1_3, CS1_4, CS5_1, CS5_2, CS5_3, CS5_4, MISO5, MOSI5, NRST, SCK5, USBDM, USBDP
- wire segments 73 -> 54
Other:
- note removed: "Spares\n"
- note removed: "Spine\n"
- moved on the sheet: C12, C13, C14, C15, C16, C17, IC2, J15, J16, J6, J7, L2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

Commit message: Updated xt-60 plug footprint
Parts:
- J8: footprint PRT-10474:SHDR2W320P716_1X2_1574X813X1588P -> xt-60:XT60
Changed lines of the file:
@@
 F 0 "J8" V 15240 1372 50  0000 R CNN
 F 1 "PRT-10474" V 15149 1372 50  0000 R CNN
-F 2 "PRT-10474:SHDR2W320P716_1X2_1574X813X1588P" H 15600 1700 50  0001 L CNN
+F 2 "xt-60:XT60" H 15600 1700 50  0001 L CNN
 F 3 "http://cdn.sparkfun.com/datasheets/Prototyping/xt60.pdf" H 15600 1600 50  0001 L CNN
 F 4 "Soldering Workstation Equipment XT60 Connectors Male/Female Pair" H 15600 1500 50  0001 L CNN "Description"
